File: _saved_droneoscillator.sch (KiCad schematic (older format))
At the start: 48 parts, among them J1 Conn_01x02, J2 Conn_01x03, Q1 BC337, Q2 BC337, Q3 BC337, Q4 BC337, U1 NE5532

Commit message: schematic bugfix, minor changes to PCB
Parts:
- D1, D2, D3, D4: footprint LEDs:LED_D5.0mm_Horizontal_O1.27mm_Z3.0mm -> LED_THT:LED_D5.0mm_Horizontal_O1.27mm_Z3.0mm
- RV1, RV2, RV3, RV4, RV5: footprint Potentiometers:Potentiometer_Alps_RK097_Single_Vertical -> Potentiometer_THT:Potentiometer_Alps_RK097_Single_Horizontal
Connections:
- net at R5.1, U1.1: now also RV5.3; no longer RV5.1
- net at C4.1, RV5.2, U1.5 (+): now also RV5.1; no longer RV5.3
Changed lines of the file:
@@
 F 0 "RV1" H 2550 1800 50  0000 C CNN
 F 1 "100K" H 2550 1700 50  0000 C CNN
-F 2 "Potentiometers:Potentiometer_Alps_RK097_Single_Vertical" H 2750 1750 50  0001 C CNN
+F 2 "Potentiometer_THT:Potentiometer_Alps_RK097_Single_Horizontal" H 2750 1750 50  0001 C CNN
 F 3 "" H 2750 1750 50  0001 C CNN
 	1    2750 1750
@@
 F 0 "D1" V 2800 2550 50  0000 C CNN
 F 1 "Red" V 2700 2550 50  0000 C CNN
-F 2 "LEDs:LED_D5.0mm_Horizontal_O1.27mm_Z3.0mm" H 2750 2700 50  0001 C CNN
+F 2 "LED_THT:LED_D5.0mm_Horizontal_O1.27mm_Z3.0mm" H 2750 2700 50  0001 C CNN
 F 3 "" H 2750 2700 50  0001 C CNN
 	1    2750 2700
@@
 F 0 "RV3" H 7100 1800 50  0000 C CNN
 F 1 "100K" H 7100 1700 50  0000 C CNN
-F 2 "Potentiometers:Potentiometer_Alps_RK097_Single_Vertical" H 7250 1750 50  0001 C CNN
+F 2 "Potentiometer_THT:Potentiometer_Alps_RK097_Single_Horizontal" H 7250 1750 50  0001 C CNN
 F 3 "" H 7250 1750 50  0001 C CNN
 	1    7250 1750
@@
 F 0 "D2" H 5100 2800 50  0000 C CNN
 F 1 "Red" H 5100 2600 50  0000 C CNN
-F 2 "LEDs:LED_D5.0mm_Horizontal_O1.27mm_Z3.0mm" H 5100 2700 50  0001 C CNN
+F 2 "LED_THT:LED_D5.0mm_Horizontal_O1.27mm_Z3.0mm" H 5100 2700 50  0001 C CNN
 F 3 "" H 5100 2700 50  0001 C CNN
 	1    5100 2700
@@
 F 0 "RV4" H 9300 1800 50  0000 C CNN
 F 1 "100K" H 9300 1700 50  0000 C CNN
-F 2 "Potentiometers:Potentiometer_Alps_RK097_Single_Vertical" H 9450 1750 50  0001 C CNN
+F 2 "Potentiometer_THT:Potentiometer_Alps_RK097_Single_Horizontal" H 9450 1750 50  0001 C CNN
 F 3 "" H 9450 1750 50  0001 C CNN
 	1    9450 1750
@@
 F 0 "D3" V 7300 2500 50  0000 C CNN
 F 1 "Red" V 7200 2500 50  0000 C CNN
-F 2 "LEDs:LED_D5.0mm_Horizontal_O1.27mm_Z3.0mm" H 7250 2700 50  0001 C CNN
+F 2 "LED_THT:LED_D5.0mm_Horizontal_O1.27mm_Z3.0mm" H 7250 2700 50  0001 C CNN
 F 3 "" H 7250 2700 50  0001 C CNN
 	1    7250 2700
@@
 F 0 "RV2" V 4925 1750 50  0000 C CNN
 F 1 "100K" V 5000 1750 50  0000 C CNN
-F 2 "Potentiometers:Potentiometer_Alps_RK097_Single_Vertical" H 5100 1750 50  0001 C CNN
+F 2 "Potentiometer_THT:Potentiometer_Alps_RK097_Single_Horizontal" H 5100 1750 50  0001 C CNN
 F 3 "" H 5100 1750 50  0001 C CNN
 	1    5100 1750
@@
 F 0 "RV5" V 2675 5150 50  0000 C CNN
 F 1 "100K" V 2750 5150 50  0000 C CNN
-F 2 "Potentiometers:Potentiometer_Alps_RK097_Single_Vertical" H 2850 5150 50  0001 C CNN
+F 2 "Potentiometer_THT:Potentiometer_Alps_RK097_Single_Horizontal" H 2850 5150 50  0001 C CNN
 F 3 "" H 2850 5150 50  0001 C CNN
 	1    2850 5150
-	0    -1   -1   0
+	0    1    -1   0
 $EndComp
 $Comp
@@
 F 0 "D4" V 9500 2550 50  0000 C CNN
 F 1 "Red" V 9400 2550 50  0000 C CNN
-F 2 "LEDs:LED_D5.0mm_Horizontal_O1.27mm_Z3.0mm" H 9450 2700 50  0001 C CNN
+F 2 "LED_THT:LED_D5.0mm_Horizontal_O1.27mm_Z3.0mm" H 9450 2700 50  0001 C CNN
 F 3 "" H 9450 2700 50  0001 C CNN
 	1    9450 2700
