File: droneoscillator.kicad_pcb (KiCad board)
At the start: 2 copper layers, 29.3 x 108.1 mm, 48 parts, among them J1 JST_XH_2, J2 JST_XH_3, Q1 BC337, Q2 BC337, Q3 BC337, Q4 BC337, U1 NE5532

Commit message: front panel changes
Parts:
- moved D4 0.51 mm to (136.0, 118.4)
- moved C10 0.38 mm to (146.2, 119.2)
- moved Q4 0.38 mm to (141.6, 121.0)
- moved D3 0.13 mm to (136.0, 96.9)
Changed lines of the file:
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@@
     (thickness 1.6)
     (drawings 10)
-    (tracks 181)
+    (tracks 179)
     (zones 0)
     (modules 48)
@@
   )
   (setup
-    (last_trace_width 0.25)
+    (last_trace_width 0.5)
     (user_trace_width 0.5)
     (user_trace_width 0.75)
@@
   )
   (module LED_THT:LED_D5.0mm_Horizontal_O1.27mm_Z3.0mm locked (layer F.Cu)
-    (at 136.017 75.452 270)
+    (at 136.017 75.438 270)
     (descr "LED, diameter 5.0mm z-position of LED center 3.0mm, 2 pins")
     (tags "LED diameter 5.0mm z-position of LED center 3.0mm 2 pins")
@@
   )
   (module LED_THT:LED_D5.0mm_Horizontal_O1.27mm_Z3.0mm locked (layer F.Cu)
-    (at 136.017 96.774 270)
+    (at 136.017 96.901 270)
     (descr "LED, diameter 5.0mm z-position of LED center 3.0mm, 2 pins")
     (tags "LED diameter 5.0mm z-position of LED center 3.0mm 2 pins")
@@
   )
   (module LED_THT:LED_D5.0mm_Horizontal_O1.27mm_Z3.0mm locked (layer F.Cu)
-    (at 136.017 118.872 270)
+    (at 136.017 118.364 270)
     (descr "LED, diameter 5.0mm z-position of LED center 3.0mm, 2 pins")
     (tags "LED diameter 5.0mm z-position of LED center 3.0mm 2 pins")
@@
   )
   (module Package_TO_SOT_THT:TO-92_Inline_Wide (layer F.Cu)
-    (at 141.605 121.38 90)
+    (at 141.605 120.999 90)
     (descr "TO-92 leads in-line, wide, drill 0.75mm (see NXP sot054_po.pdf)")
     (tags "to-92 sc-43 sc-43a sot54 PA33 transistor")
@@
   )
   (module Capacitor_THT:CP_Radial_D4.0mm_P2.00mm (layer F.Cu)
-    (at 146.177 119.602 270)
+    (at 146.177 119.221 270)
     (descr "CP, Radial series, Radial, pin pitch=2.00mm, , diameter=4mm, Electrolytic Capacitor")
     (tags "CP Radial series Radial pin pitch 2.00mm  diameter 4mm Electrolytic Capacitor")
@@
   (segment (start 136.13 105) (end 136.13 108.38) (width 0.5) (layer B.Cu) (net 22))
   (segment (start 136.5 108.75) (end 136.5 111.25) (width 0.5) (layer B.Cu) (net 22))
-  (segment (start 136.5 111.25) (end 140.46 111.25) (width 0.5) (layer B.Cu) (net 22))
-  (segment (start 141.355 112.145) (end 141.355 116.411) (width 0.5) (layer B.Cu) (net 22))
-  (segment (start 140.46 111.25) (end 141.355 112.145) (width 0.5) (layer B.Cu) (net 22))
-  (segment (start 146.177 116.967) (end 146.177 119.602) (width 0.5) (layer B.Cu) (net 22))
-  (segment (start 141.605 116.3) (end 145.51 116.3) (width 0.5) (layer B.Cu) (net 22))
-  (segment (start 145.51 116.3) (end 146.177 116.967) (width 0.5) (layer B.Cu) (net 22))
-  (segment (start 141.827 121.602) (end 141.605 121.38) (width 0.5) (layer B.Cu) (net 23))
-  (segment (start 146.177 121.602) (end 141.827 121.602) (width 0.5) (layer B.Cu) (net 23))
-  (segment (start 141.605 121.38) (end 138.049 121.38) (width 0.5) (layer B.Cu) (net 23))
-  (segment (start 137.321792 121.38) (end 138.049 121.38) (width 0.5) (layer B.Cu) (net 23))
-  (segment (start 136.017 121.412) (end 137.289792 121.412) (width 0.5) (layer B.Cu) (net 23))
-  (segment (start 137.289792 121.412) (end 137.321792 121.38) (width 0.5) (layer B.Cu) (net 23))
+  (segment (start 146.177 116.586) (end 146.177 119.221) (width 0.5) (layer B.Cu) (net 22))
+  (segment (start 141.605 115.919) (end 145.51 115.919) (width 0.5) (layer B.Cu) (net 22))
+  (segment (start 145.51 115.919) (end 146.177 116.586) (width 0.5) (layer B.Cu) (net 22))
+  (segment (start 140.46 111.25) (end 136.5 111.25) (width 0.5) (layer B.Cu) (net 22))
+  (segment (start 141.605 115.919) (end 141.605 112.395) (width 0.5) (layer B.Cu) (net 22))
+  (segment (start 141.605 112.395) (end 140.46 111.25) (width 0.5) (layer B.Cu) (net 22))
+  (segment (start 141.827 121.221) (end 141.605 120.999) (width 0.5) (layer B.Cu) (net 23))
+  (segment (start 146.177 121.221) (end 141.827 121.221) (width 0.5) (layer B.Cu) (net 23))
+  (segment (start 141.51 120.904) (end 141.605 120.999) (width 0.5) (layer B.Cu) (net 23))
+  (segment (start 136.017 120.904) (end 141.51 120.904) (width 0.5) (layer B.Cu) (net 23))
   (segment (start 148.848 102.854) (end 148.848 103.98537) (width 0.5) (layer B.Cu) (net 24))
   (segment (start 148.848 107.426) (end 148.848 104.124) (width 0.5) (layer B.Cu) (net 24))

Commit message: updated BOM + component notes
Parts:
- D1, D2, D3, D4: value Red -> 5mm red
- J1: value JST_XH_2 -> NF
Changed lines of the file:
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@@
       (effects (font (size 1 1) (thickness 0.15)))
     )
-    (fp_text value JST_XH_2 (at 1.25 4.6) (layer F.Fab)
+    (fp_text value NF (at 1.25 4.6) (layer F.Fab)
       (effects (font (size 1 1) (thickness 0.15)))
     )
@@
       (effects (font (size 1 1) (thickness 0.15)))
     )
-    (fp_text value Red (at 1.27 10.93 270) (layer F.Fab)
+    (fp_text value "5mm red" (at 1.27 10.93 270) (layer F.Fab)
       (effects (font (size 1 1) (thickness 0.15)))
     )
@@
       (effects (font (size 1 1) (thickness 0.15)))
     )
-    (fp_text value Red (at 1.27 10.93 270) (layer F.Fab)
+    (fp_text value "5mm red" (at 1.27 10.93 270) (layer F.Fab)
       (effects (font (size 1 1) (thickness 0.15)))
     )
@@
       (effects (font (size 1 1) (thickness 0.15)))
     )
-    (fp_text value Red (at 1.27 10.93 270) (layer F.Fab)
+    (fp_text value "5mm red" (at 1.27 10.93 270) (layer F.Fab)
       (effects (font (size 1 1) (thickness 0.15)))
     )
@@
       (effects (font (size 1 1) (thickness 0.15)))
     )
-    (fp_text value Red (at 1.27 10.93 270) (layer F.Fab)
-      (effects (font (size 1 1) (thickness 0.15)))
-    )
+    (fp_text value "5mm red" (at 1.27 10.93 270) (layer F.Fab)
+      (effects (font (size 1 1) (thickness 0.15)))
+    )
